Commit message: implemented merge requirements, added model type .2 to modelparameters

File: data/trajectories/design_A.0/model_1.2/acrobot/dircol/trajopt/20231201-150842/acrobot.urdf (robot description, URDF)
Before this commit: robot acrobot, 4 links, 4 joints
Joints:
- joint Joint2: limit lower=-3.1415926 upper=3.1415926 effort=6.0 velocity=20 -> lower=-3.1415926 upper=3.1415926 effort=10.0 velocity=20
